File: tech_safari_data_logger/tech_safari_data_logger.brd (EAGLE design)
At the start: 90.2 x 52.1 mm, 11 parts, among them U1 TEENSY_3.2_NB_LP

Commit message: swapped GPS/SD positions for no overlap
Parts:
- moved SD 29.2 mm to (41.9, 22.9)
- moved ULTIMATEGPS 28.7 mm to (71.1, 20.3)
Routing:
- net SDCD: track 41.7 -> 12.8 mm
- net SDCS: track 39.2 -> 12.8 mm
- net SDDI: track 36.7 -> 12.8 mm
- net SDDO: track 35.3 -> 12.8 mm
- net GPSTX: track 5.08 -> 25.5 mm
- net GPSRX: track 5.08 -> 25.5 mm
- net SDCLK: track 36.8 -> 28.7 mm
- net +3V3: track 223.1 -> 227.6 mm

Commit message: cleaned up layout of sch and brd
Parts:
- removed R4: (no value), rcl:0207/10
- added POT: (no value), personal:POTENTIOMETER_THRU
- R1: value (none) -> 220; device personal:POTENTIOMETER_THRU -> rcl:0207/10
- R2, R3: value (none) -> 220
- moved R1 72.5 mm to (24.1, 40.6), turned to 180 degrees
- moved R2 15.3 mm to (24.1, 38.1)
- moved R3 15.3 mm to (24.1, 35.6)
- moved BME680 13.7 mm to (59.7, 35.6)
- moved ULTIMATEGPS 13.7 mm to (59.7, 12.7)
- moved RGBLED 13.7 mm to (14.0, 39.4)
- moved U1 13.7 mm to (44.5, 22.9)
- moved COINCELL 13.7 mm to (16.5, 17.8)
- moved LIPO 13.7 mm to (33.0, 47.0)
- moved SD 13.7 mm to (30.5, 15.2)
Connections:
- net +3V3: now also POT.3; no longer R1.3
- net AGND: now also POT.1; no longer R1.1
- net LED0: now also R1.1; no longer R2.1
- net LED1: now also R2.1; no longer R3.1
- net LED2: now also R3.1; no longer R4.1
- net N$5: now also R1.2; no longer R2.2
- net N$6: now also R2.2; no longer R3.2
- net N$7: now also R3.2; no longer R4.2
- net POT: now also POT.2; no longer R1.2
Routing:
- net +3V3: track 227.6 -> 222.2 mm
- net POT: track 32.3 -> 28.5 mm
- net AGND: track 31.2 -> 27.4 mm
Other:
- board size 90.2 x 52.1 mm -> 91.4 x 52.1 mm
- board text added: "Note: run wire from Coin+ to Vbat on Teensy"
- board text added: "Tech Safari Data Logger"
