File: tech_safari_data_logger/tech_safari_data_logger.sch (EAGLE design)
At the start: 11 parts, among them U1 TEENSY_3.2_NB_LP

Commit message: cleaned up layout of sch and brd
Parts:
- removed R4: (no value), rcl:R-EU_0207/10
- added POT: POTENTIOMETER_THRU, personal:POTENTIOMETER_THRU
- R1: value POTENTIOMETER_THRU -> 220; device personal:POTENTIOMETER_THRU -> rcl:R-EU_0207/10
- R2, R3: value (none) -> 220
Connections:
- net +3V3: now also POT.3; no longer R1.3
- net AGND: now also POT.1; no longer R1.1
- net LED0: now also R1.1; no longer R2.1
- net LED1: now also R2.1; no longer R3.1
- net LED2: now also R3.1; no longer R4.1
- net N$5: now also R1.2; no longer R2.2
- net N$6: now also R2.2; no longer R3.2
- net N$7: now also R3.2; no longer R4.2
- net POT: now also POT.2; no longer R1.2
Other:
- note added: "1 of 1"
- note added: "2"
- note added: "American University Computer Science Tech Safari 2018"
- note added: "Breakout boards"
- note added: "I/O"
- note added: "Microcontroller"
- note added: "Power"
- moved on the sheet: BME680, COINCELL, LIPO, R2, R3, RGBLED, SD, U1, ULTIMATEGPS
